Commit message: added camera to robot and took care of footage visualization through openCV

File: alberto_description/urdf/alberto.gazebo.xacro (robot description, xacro)
@@ -1,6 +1,6 @@
 <?xml version="1.0"?>
 <robot name="alberto" xmlns:xacro="http://ros.org/wiki/xacro">
-  <xacro:arg name="laser_visual" default="false"/>
-  <xacro:arg name="imu_visual"   default="false"/>
+  <xacro:arg name="laser_visual" default="false" />
+  <xacro:arg name="imu_visual" default="false" />
   <gazebo reference="base_link">
     <material>Gazebo/DarkGrey</material>
@@ -124,3 +124,40 @@
     </sensor>
   </gazebo>
+  <!-- camera -->
+  <gazebo reference="camera_link">
+    <sensor type="camera" name="camera1">
+      <update_rate>30.0</update_rate>
+      <camera name="head">
+        <horizontal_fov>1.3962634</horizontal_fov>
+        <image>
+          <width>800</width>
+          <height>800</height>
+          <format>R8G8B8</format>
+        </image>
+        <clip>
+          <near>0.02</near>
+          <far>300</far>
+        </clip>
+        <noise>
+          <type>gaussian</type>
+          <mean>0.0</mean>
+          <stddev>0.007</stddev>
+        </noise>
+      </camera>
+      <plugin name="camera_controller" filename="libgazebo_ros_camera.so">
+        <alwaysOn>true</alwaysOn>
+        <updateRate>0.0</updateRate>
+        <cameraName>rrbot/camera1</cameraName>
+        <imageTopicName>image_raw</imageTopicName>
+        <cameraInfoTopicName>camera_info</cameraInfoTopicName>
+        <frameName>camera_link</frameName>
+        <hackBaseline>0.07</hackBaseline>
+        <distortionK1>0.0</distortionK1>
+        <distortionK2>0.0</distortionK2>
+        <distortionK3>0.0</distortionK3>
+        <distortionT1>0.0</distortionT1>
+        <distortionT2>0.0</distortionT2>
+      </plugin>
+    </sensor>
+  </gazebo>
 </robot>

File: alberto_description/urdf/alberto.urdf.xacro (robot description, xacro)
@@ -1,52 +1,55 @@
-<?xml version="1.0" ?>
+<?xml version="1.0"?>
 <robot name="alberto" xmlns:xacro="http://ros.org/wiki/xacro">
-  <xacro:include filename="$(find alberto_description)/urdf/common_properties.xacro"/>
-  <xacro:include filename="$(find alberto_description)/urdf/alberto.gazebo.xacro"/>
-  <link name="base_footprint"/>
+  <xacro:include filename="$(find alberto_description)/urdf/common_properties.xacro" />
+  <xacro:include filename="$(find alberto_description)/urdf/alberto.gazebo.xacro" />
+  <xacro:property name="camera_link" value="0.05" />
+  <link name="base_footprint" />
   <joint name="base_joint" type="fixed">
-    <parent link="base_footprint"/>
-    <child link="base_link"/>
-    <origin xyz="0.0 0.0 0.010" rpy="0 0 0"/>
+    <parent link="base_footprint" />
+    <child link="base_link" />
+    <origin xyz="0.0 0.0 0.010" rpy="0 0 0" />
   </joint>
   <link name="base_link">
     <visual>
-      <origin xyz="-0.032 0 0.0" rpy="0 0 0"/>
+      <origin xyz="-0.032 0 0.0" rpy="0 0 0" />
       <geometry>
-        <mesh filename="package://turtlebot3_description/meshes/bases/burger_base.stl" scale="0.001 0.001 0.001"/>
+        <mesh filename="package://turtlebot3_description/meshes/bases/burger_base.stl"
+          scale="0.001 0.001 0.001" />
       </geometry>
-      <material name="light_black"/>
+      <material name="light_black" />
     </visual>
     <collision>
-      <origin xyz="-0.032 0 0.070" rpy="0 0 0"/>
+      <origin xyz="-0.032 0 0.070" rpy="0 0 0" />
       <geometry>
-        <box size="0.140 0.140 0.143"/>
+        <box size="0.140 0.140 0.143" />
       </geometry>
     </collision>
     <inertial>
-      <origin xyz="0 0 0" rpy="0 0 0"/>
-      <mass value="8.2573504e-01"/>
+      <origin xyz="0 0 0" rpy="0 0 0" />
+      <mass value="8.2573504e-01" />
       <inertia ixx="2.2124416e-03" ixy="-1.2294101e-05" ixz="3.4938785e-05"
-               iyy="2.1193702e-03" iyz="-5.0120904e-06"
-               izz="2.0064271e-03" />
+        iyy="2.1193702e-03" iyz="-5.0120904e-06"
+        izz="2.0064271e-03" />
     </inertial>
   </link>
   <joint name="wheel_left_joint" type="continuous">
-    <parent link="base_link"/>
-    <child link="wheel_left_link"/>
-    <origin xyz="0.0 0.08 0.023" rpy="-1.57 0 0"/>
-    <axis xyz="0 0 1"/>
+    <parent link="base_link" />
+    <child link="wheel_left_link" />
+    <origin xyz="0.0 0.08 0.023" rpy="-1.57 0 0" />
+    <axis xyz="0 0 1" />
   </joint>
   <link name="wheel_left_link">
     <visual>
-      <origin xyz="0 0 0" rpy="1.57 0 0"/>
+      <origin xyz="0 0 0" rpy="1.57 0 0" />
       <geometry>
-        <mesh filename="package://turtlebot3_description/meshes/wheels/left_tire.stl" scale="0.001 0.001 0.001"/>
+        <mesh filename="package://turtlebot3_description/meshes/wheels/left_tire.stl"
+          scale="0.001 0.001 0.001" />
       </geometry>
-      <material name="dark"/>
+      <material name="dark" />
     </visual>
     <collision>
-      <origin xyz="0 0 0" rpy="0 0 0"/>
+      <origin xyz="0 0 0" rpy="0 0 0" />
       <geometry>
-        <cylinder length="0.018" radius="0.033"/>
+        <cylinder length="0.018" radius="0.033" />
       </geometry>
     </collision>
@@ -55,26 +58,27 @@
       <mass value="2.8498940e-02" />
       <inertia ixx="1.1175580e-05" ixy="-4.2369783e-11" ixz="-5.9381719e-09"
-               iyy="1.1192413e-05" iyz="-1.4400107e-11"
-               izz="2.0712558e-05" />
-      </inertial>
+        iyy="1.1192413e-05" iyz="-1.4400107e-11"
+        izz="2.0712558e-05" />
+    </inertial>
   </link>
   <joint name="wheel_right_joint" type="continuous">
-    <parent link="base_link"/>
-    <child link="wheel_right_link"/>
-    <origin xyz="0.0 -0.080 0.023" rpy="-1.57 0 0"/>
-    <axis xyz="0 0 1"/>
+    <parent link="base_link" />
+    <child link="wheel_right_link" />
+    <origin xyz="0.0 -0.080 0.023" rpy="-1.57 0 0" />
+    <axis xyz="0 0 1" />
   </joint>
   <link name="wheel_right_link">
     <visual>
-      <origin xyz="0 0 0" rpy="1.57 0 0"/>
+      <origin xyz="0 0 0" rpy="1.57 0 0" />
       <geometry>
-        <mesh filename="package://turtlebot3_description/meshes/wheels/right_tire.stl" scale="0.001 0.001 0.001"/>
+        <mesh filename="package://turtlebot3_description/meshes/wheels/right_tire.stl"
+          scale="0.001 0.001 0.001" />
       </geometry>
-      <material name="dark"/>
+      <material name="dark" />
     </visual>
     <collision>
-      <origin xyz="0 0 0" rpy="0 0 0"/>
+      <origin xyz="0 0 0" rpy="0 0 0" />
       <geometry>
-        <cylinder length="0.018" radius="0.033"/>
+        <cylinder length="0.018" radius="0.033" />
       </geometry>
     </collision>
@@ -83,18 +87,18 @@
       <mass value="2.8498940e-02" />
       <inertia ixx="1.1175580e-05" ixy="-4.2369783e-11" ixz="-5.9381719e-09"
-               iyy="1.1192413e-05" iyz="-1.4400107e-11"
-               izz="2.0712558e-05" />
-      </inertial>
+        iyy="1.1192413e-05" iyz="-1.4400107e-11"
+        izz="2.0712558e-05" />
+    </inertial>
   </link>
   <joint name="caster_back_joint" type="fixed">
-    <parent link="base_link"/>
-    <child link="caster_back_link"/>
-    <origin xyz="-0.081 0 -0.004" rpy="-1.57 0 0"/>
+    <parent link="base_link" />
+    <child link="caster_back_link" />
+    <origin xyz="-0.081 0 -0.004" rpy="-1.57 0 0" />
   </joint>
   <link name="caster_back_link">
     <collision>
-      <origin xyz="0 0.001 0" rpy="0 0 0"/>
+      <origin xyz="0 0.001 0" rpy="0 0 0" />
       <geometry>
-        <box size="0.030 0.009 0.020"/>
+        <box size="0.030 0.009 0.020" />
       </geometry>
     </collision>
@@ -103,31 +107,32 @@
       <mass value="0.005" />
       <inertia ixx="0.001" ixy="0.0" ixz="0.0"
-               iyy="0.001" iyz="0.0"
-               izz="0.001" />
+        iyy="0.001" iyz="0.0"
+        izz="0.001" />
     </inertial>
   </link>
   <joint name="imu_joint" type="fixed">
-    <parent link="base_link"/>
-    <child link="imu_link"/>
-    <origin xyz="-0.032 0 0.068" rpy="0 0 0"/>
+    <parent link="base_link" />
+    <child link="imu_link" />
+    <origin xyz="-0.032 0 0.068" rpy="0 0 0" />
   </joint>
-  <link name="imu_link"/>
+  <link name="imu_link" />
   <joint name="scan_joint" type="fixed">
-    <parent link="base_link"/>
-    <child link="base_scan"/>
-    <origin xyz="-0.032 0 0.172" rpy="0 0 0"/>
+    <parent link="base_link" />
+    <child link="base_scan" />
+    <origin xyz="-0.032 0 0.172" rpy="0 0 0" />
   </joint>
   <link name="base_scan">
     <visual>
-      <origin xyz="0 0 0.0" rpy="0 0 0"/>
+      <origin xyz="0 0 0.0" rpy="0 0 0" />
       <geometry>
-        <mesh filename="package://turtlebot3_description/meshes/sensors/lds.stl" scale="0.001 0.001 0.001"/>
+        <mesh filename="package://turtlebot3_description/meshes/sensors/lds.stl"
+          scale="0.001 0.001 0.001" />
       </geometry>
-      <material name="dark"/>
+      <material name="dark" />
     </visual>
     <collision>
-      <origin xyz="0.015 0 -0.0065" rpy="0 0 0"/>
+      <origin xyz="0.015 0 -0.0065" rpy="0 0 0" />
       <geometry>
-        <cylinder length="0.0315" radius="0.055"/>
+        <cylinder length="0.0315" radius="0.055" />
       </geometry>
     </collision>
@@ -136,6 +141,33 @@
       <origin xyz="0 0 0" />
       <inertia ixx="0.001" ixy="0.0" ixz="0.0"
-               iyy="0.001" iyz="0.0"
-               izz="0.001" />
+        iyy="0.001" iyz="0.0"
+        izz="0.001" />
+    </inertial>
+  </link>
+  <joint name="camera_joint" type="fixed">
+    <axis xyz="0 1 0" />
+    <origin xyz="0 0 0.5" rpy="0 0 0" />
+    <parent link="base_link" />
+    <child link="camera_link" />
+  </joint>
+  <!-- Camera -->
+  <link name="camera_link">
+    <collision>
+      <origin xyz="0 0 0" rpy="0 0 0" />
+      <geometry>
+        <box size="${camera_link} ${camera_link} ${camera_link}" />
+      </geometry>
+    </collision>
+    <visual>
+      <origin xyz="0 0 0" rpy="0 0 0" />
+      <geometry>
+        <box size="${camera_link} ${camera_link} ${camera_link}" />
+      </geometry>
+      <material name="red" />
+    </visual>
+    <inertial>
+      <mass value="1e-5" />
+      <origin xyz="0 0 0" rpy="0 0 0" />
+      <inertia ixx="1e-6" ixy="0" ixz="0" iyy="1e-6" iyz="0" izz="1e-6" />
     </inertial>
   </link>

Commit message: figuring out if people are real or pictures

File: alberto_description/urdf/alberto.gazebo.xacro (robot description, xacro)
@@ -124,6 +124,6 @@
     </sensor>
   </gazebo>
-  <!-- camera -->
-  <gazebo reference="camera_link">
+  <!-- RGB camera -->
+  <!-- <gazebo reference="camera_link">
     <sensor type="camera" name="camera1">
       <update_rate>30.0</update_rate>
@@ -160,4 +160,46 @@
       </plugin>
     </sensor>
+  </gazebo> -->
+  <!-- depth camera -->
+  <gazebo reference="depth_camera_link">
+    <sensor name="depth_camera_link_camera" type="depth">
+      <update_rate>20</update_rate>
+      <camera>
+        <horizontal_fov>1.047198</horizontal_fov>
+        <image>
+          <width>640</width>
+          <height>480</height>
+          <format>R8G8B8</format>
+        </image>
+        <clip>
+          <near>0.05</near>
+          <far>10</far>
+        </clip>
+      </camera>
+      <plugin name="depth_camera_link_controller" filename="libgazebo_ros_openni_kinect.so">
+        <baseline>0.2</baseline>
+        <alwaysOn>true</alwaysOn>
+        <updateRate>1.0</updateRate>
+        <cameraName>depth_camera_ir</cameraName>
+        <imageTopicName>/depth_camera/color/image_raw</imageTopicName>
+        <cameraInfoTopicName>/depth_camera/color/camera_info</cameraInfoTopicName>
+        <depthImageTopicName>/depth_camera/depth/image_raw</depthImageTopicName>
+        <depthImageInfoTopicName>/depth_camera/depth/camera_info</depthImageInfoTopicName>
+        <pointCloudTopicName>/depth_camera/depth/points</pointCloudTopicName>
+        <frameName>depth_camera_link</frameName>
+        <pointCloudCutoff>0.5</pointCloudCutoff>
+        <pointCloudCutoffMax>10</pointCloudCutoffMax>
+        <distortionK1>0.00000001</distortionK1>
+        <distortionK2>0.00000001</distortionK2>
+        <distortionK3>0.00000001</distortionK3>
+        <distortionT1>0.00000001</distortionT1>
+        <distortionT2>0.00000001</distortionT2>
+        <CxPrime>0</CxPrime>
+        <Cx>0</Cx>
+        <Cy>0</Cy>
+        <focalLength>0</focalLength>
+        <hackBaseline>0</hackBaseline>
+      </plugin>
+    </sensor>
   </gazebo>
 </robot>

File: alberto_description/urdf/alberto.urdf.xacro (robot description, xacro)
@@ -145,12 +145,12 @@
     </inertial>
   </link>
-  <joint name="camera_joint" type="fixed">
+  <joint name="depth_camera_joint" type="fixed">
     <axis xyz="0 1 0" />
     <origin xyz="0 0 0.5" rpy="0 0 0" />
     <parent link="base_link" />
-    <child link="camera_link" />
+    <child link="depth_camera_link" />
   </joint>
-  <!-- Camera -->
-  <link name="camera_link">
+  <!-- depth camera -->
+  <link name="depth_camera_link">
     <collision>
       <origin xyz="0 0 0" rpy="0 0 0" />
